File: A.E.K.brd (EAGLE design)
At the start: 68.6 x 53.3 mm, 7 parts

Commit message: schemetics change
remove unroute pin
Connections:
- removed net IOREF: B_L_JP2.7
- removed net N$23: B_L_JP2.8
- removed net N$24: U$1.RST1
- removed net N$40: U$1.A7
- removed net N$41: U$1.A6
- removed net N$50: U$1.D13
- removed net SCL: T_L_JP4.1
- removed net SDA: T_L_JP4.2
- net D13: now also U$1.D13
Changed lines of the file:
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@@
 <drawing>
 <settings>
-<setting alwaysvectorfont="yes"/>
+<setting alwaysvectorfont="no"/>
 <setting verticaltext="up"/>
 </settings>
@@
 <signal name="D13">
 <contactref element="T_L_JP4" pad="5"/>
+<contactref element="U$1" pad="D13"/>
+<wire x1="2.54" y1="10.16" x2="28.956" y2="50.8" width="0" layer="19" extent="1-1"/>
 </signal>
 <signal name="AREF">
@@
 <wire x1="7.62" y1="10.16" x2="23.876" y2="50.8" width="0" layer="19" extent="1-1"/>
 </signal>
-<signal name="SDA">
-<contactref element="T_L_JP4" pad="2"/>
-</signal>
-<signal name="SCL">
-<contactref element="T_L_JP4" pad="1"/>
-</signal>
 <signal name="3.3V">
 <contactref element="B_L_JP2" pad="5"/>
 <contactref element="U$1" pad="3.3V"/>
 <wire x1="5.08" y1="10.16" x2="35.56" y2="2.54" width="0" layer="19" extent="1-1"/>
-</signal>
-<signal name="IOREF">
-<contactref element="B_L_JP2" pad="7"/>
-</signal>
-<signal name="N$23">
-<contactref element="B_L_JP2" pad="8"/>
-</signal>
-<signal name="N$24">
-<contactref element="U$1" pad="RST1"/>
 </signal>
 <signal name="D8">
@@
 <wire x1="46.355" y1="12.7" x2="30.48" y2="10.16" width="0" layer="19" extent="1-1"/>
 </signal>
-<signal name="N$40">
-<contactref element="U$1" pad="A7"/>
-</signal>
-<signal name="N$41">
-<contactref element="U$1" pad="A6"/>
-</signal>
-<signal name="N$50">
-<contactref element="U$1" pad="D13"/>
-</signal>
 <signal name="A0">
